File: kicad/Treg.kicad_sch (KiCad schematic)
At the start: 44 parts, among them J1 Conn_01x02, J2 Conn_01x02, J3 Conn_01x02, J4 Conn_01x02, J5 Conn_01x02, J7 Conn_01x07, J8 Conn_01x07, J9 Conn_01x02, U1 PMW3360, U2 TPS73601DBV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

Commit message: add caps, jp
Parts:
- removed U1: PMW3360, footprint:PMW3360, symbol PMW3360:PMW3360
- added C7: 100nF, Capacitor_SMD:C_0603_1608Metric, symbol Device:C_Small
- added C8: 10uF, Capacitor_SMD:C_0603_1608Metric, symbol Device:C_Small
- added JP1: SolderJumper_2_Bridged, Jumper:SolderJumper-2_P1.3mm_Bridged_RoundedPad1.0x1.5mm, symbol Jumper:SolderJumper_2_Bridged
- added U1: PMW3360, footprint:PMW3360, symbol pmw3360:pmw3360
- C4, C6: value 100nF -> 10uF
Connections:
- net 1V9: now also C7.1, C8.1, U1.4 (VDD)
- net 3V3: now also U1.5 (VDDIO)
- net GND: now also C7.2, C8.2, JP1.2 (B), U1.8 (GND)
- net MISO: now also U1.12 (MISO)
- net MOSI: now also U1.11 (MOSI)
- net MOTION: now also U1.9 (MOTION)
- net NRESET: now also U1.7 (nRESET)
- net SCLK: now also U1.10 (SCLK)
- net at C1.1, C2.1: now also U1.3 (VDDPIX)
- net at R1.2: now also U1.15 (LED_P)
- net nc: now reaches J7.1 (Pin_1)
- net nc: now also U3.1 (GPIO0_A0_D0)
- new net NCS: JP1.1 (A), U1.13 (nCS)
- no-connect marks 10 -> 8
Other:
- moved on the sheet: C1, C11, C12, C13, C14, C2, H1, H2, H3, H4, R1, R2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

Commit message: add C9
Parts:
- added C9: 100nF, Capacitor_SMD:C_0603_1608Metric, symbol Device:C_Small
Connections:
- net 3V3: now also C9.1
- net GND: now also C9.2
Other:
- moved on the sheet: C3, C4
Changed lines of the file:
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@@
 	)
 	(junction
-		(at 66.04 27.94)
+		(at 55.88 27.94)
 		(diameter 0)
 		(color 0 0 0 0)
@@
 	)
 	(junction
+		(at 66.04 27.94)
+		(diameter 0)
+		(color 0 0 0 0)
+	)
+	(junction
 		(at 53.34 119.38)
 		(diameter 0)
@@
 	)
 	(junction
+		(at 66.04 22.86)
+		(diameter 0)
+		(color 0 0 0 0)
+	)
+	(junction
 		(at 127 110.49)
 		(diameter 0)
@@
 	)
 	(junction
-		(at 66.04 22.86)
+		(at 55.88 22.86)
 		(diameter 0)
 		(color 0 0 0 0)
@@
 	(wire
 		(pts
-			(xy 66.04 27.94) (xy 76.2 27.94)
+			(xy 55.88 27.94) (xy 66.04 27.94)
 		)
 		(stroke
@@
 	(wire
 		(pts
+			(xy 66.04 27.94) (xy 76.2 27.94)
+		)
+		(stroke
+			(width 0)
+			(type default)
+		)
+	)
+	(wire
+		(pts
 			(xy 137.16 107.95) (xy 137.16 110.49)
 		)
@@
 	(wire
 		(pts
+			(xy 55.88 22.86) (xy 66.04 22.86)
+		)
+		(stroke
+			(width 0)
+			(type default)
+		)
+	)
+	(wire
+		(pts
 			(xy 66.04 22.86) (xy 76.2 22.86)
 		)
@@
 	(symbol
 		(lib_id "power:VDD")
-		(at 66.04 22.86 0)
+		(at 55.88 22.86 0)
 		(unit 1)
 		(exclude_from_sim no)
@@
 		(fields_autoplaced yes)
 		(property "Reference" "#PWR07"
-			(at 66.04 26.67 0)
+			(at 55.88 26.67 0)
 			(effects
 				(font
@@
 		)
 		(property "Value" "3V3"
-			(at 66.04 17.78 0)
+			(at 55.88 17.78 0)
 			(effects
 				(font
@@
 		)
 		(property "Footprint" ""
-			(at 66.04 22.86 0)
+			(at 55.88 22.86 0)
 			(effects
 				(font
@@
 		)
 		(property "Datasheet" ""
-			(at 66.04 22.86 0)
+			(at 55.88 22.86 0)
 			(effects
 				(font
@@
 		)
 		(property "Description" "Power symbol creates a global label with name \"VDD\""
-			(at 66.04 22.86 0)
+			(at 55.88 22.86 0)
 			(effects
 				(font
@@
 	(symbol
 		(lib_id "Device:C_Small")
-		(at 66.04 25.4 0)
+		(at 55.88 25.4 0)
 		(mirror y)
 		(unit 1)
@@
 		(dnp no)
 		(property "Reference" "C3"
-			(at 63.5 24.1362 0)
+			(at 53.34 24.1362 0)
 			(effects
 				(font
@@
 		)
 		(property "Value" "100nF"
-			(at 63.5 26.6762 0)
+			(at 53.34 26.6762 0)
 			(effects
 				(font
@@
 		)
 		(property "Footprint" "Capacitor_SMD:C_0603_1608Metric"
-			(at 66.04 25.4 0)
+			(at 55.88 25.4 0)
 			(effects
 				(font
@@
 		)
 		(property "Datasheet" "~"
-			(at 66.04 25.4 0)
+			(at 55.88 25.4 0)
 			(effects
 				(font
@@
 		)
 		(property "Description" "Unpolarized capacitor, small symbol"
-			(at 66.04 25.4 0)
+			(at 55.88 25.4 0)
 			(effects
 				(font
@@
 	(symbol
 		(lib_id "power:GND")
-		(at 66.04 27.94 0)
+		(at 55.88 27.94 0)
 		(unit 1)
 		(exclude_from_sim no)
@@
 		(fields_autoplaced yes)
 		(property "Reference" "#PWR08"
-			(at 66.04 34.29 0)
+			(at 55.88 34.29 0)
 			(effects
 				(font
@@
 		)
 		(property "Value" "GND"
-			(at 66.04 33.02 0)
+			(at 55.88 33.02 0)
 			(effects
 				(font
@@
 		)
 		(property "Footprint" ""
-			(at 66.04 27.94 0)
+			(at 55.88 27.94 0)
 			(effects
 				(font
@@
 		)
 		(property "Datasheet" ""
-			(at 66.04 27.94 0)
+			(at 55.88 27.94 0)
 			(effects
 				(font
@@
 		)
 		(property "Description" "Power symbol creates a global label with name \"GND\" , ground"
-			(at 66.04 27.94 0)
+			(at 55.88 27.94 0)
 			(effects
 				(font
@@
 	)
 	(symbol
+		(lib_id "Device:C_Small")
+		(at 76.2 25.4 0)
+		(mirror y)
+		(unit 1)
+		(exclude_from_sim no)
+		(in_bom yes)
+		(on_board yes)
+		(dnp no)
+		(property "Reference" "C9"
+			(at 73.66 24.1362 0)
+			(effects
+				(font
+					(size 1.27 1.27)
+				)
+				(justify left)
+			)
+		)
+		(property "Value" "100nF"
+			(at 73.66 26.6762 0)
+			(effects
+				(font
+					(size 1.27 1.27)
+				)
+				(justify left)
+			)
+		)
+		(property "Footprint" "Capacitor_SMD:C_0603_1608Metric"
+			(at 76.2 25.4 0)
+			(effects
+				(font
+					(size 1.27 1.27)
+				)
+				(hide yes)
+			)
+		)
+		(property "Datasheet" "~"
+			(at 76.2 25.4 0)
+			(effects
+				(font
+					(size 1.27 1.27)
+				)
+				(hide yes)
+			)
+		)
+		(property "Description" "Unpolarized capacitor, small symbol"
+			(at 76.2 25.4 0)
+			(effects
+				(font
+					(size 1.27 1.27)
+				)
+				(hide yes)
+			)
+		)
+		(pin "1"
+		)
+		(pin "2"
+		)
+		(instances
+			(project "Treg"
+				(path "/cc713380-d5d4-4611-b364-320b19da6c16"
+					(reference "C9")
+					(unit 1)
+				)
+			)
+		)
+	)
+	(symbol
 		(lib_id "Seeed_Studio_XIAO_Series:XIAO-ESP32-C6-SMD")
 		(at 171.45 44.45 0)
@@
 	(symbol
 		(lib_id "Device:C_Small")
-		(at 76.2 25.4 0)
+		(at 66.04 25.4 0)
 		(mirror y)
 		(unit 1)
@@
 		(dnp no)
 		(property "Reference" "C4"
-			(at 73.66 24.1362 0)
+			(at 63.5 24.1362 0)
 			(effects
 				(font
@@
 		)
 		(property "Value" "10uF"
-			(at 73.66 26.6762 0)
+			(at 63.5 26.6762 0)
 			(effects
 				(font
@@
 		)
 		(property "Footprint" "Capacitor_SMD:C_0603_1608Metric"
-			(at 76.2 25.4 0)
+			(at 66.04 25.4 0)
 			(effects
 				(font
@@
 		)
 		(property "Datasheet" "~"
-			(at 76.2 25.4 0)
+			(at 66.04 25.4 0)
 			(effects
 				(font
@@
 		)
 		(property "Description" "Unpolarized capacitor, small symbol"
-			(at 76.2 25.4 0)
+			(at 66.04 25.4 0)
 			(effects
 				(font

Commit message: removed jp1
Parts:
- removed JP1: SolderJumper_2_Bridged, Jumper:SolderJumper-2_P1.3mm_Bridged_RoundedPad1.0x1.5mm, symbol Jumper:SolderJumper_2_Bridged
Connections:
- net NCS is gone; now on net GND: U1.13 (nCS)
Changed lines of the file:
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@@
 		)
 	)
-	(global_label "NCS"
-		(shape input)
-		(at 59.69 85.09 180)
-		(fields_autoplaced yes)
-		(effects
-			(font
-				(size 1.27 1.27)
-			)
-			(justify right)
-		)
-		(property "Intersheetrefs" "${INTERSHEET_REFS}"
-			(at 52.8948 85.09 0)
-			(effects
-				(font
-					(size 1.27 1.27)
-				)
-				(justify right)
-				(hide yes)
-			)
-		)
-	)
 	(global_label "DSW4"
 		(shape input)
@@
 		)
 	)
-	(global_label "NCS"
-		(shape input)
-		(at 73.66 60.96 0)
-		(fields_autoplaced yes)
-		(effects
-			(font
-				(size 1.27 1.27)
-			)
-			(justify left)
-		)
-		(property "Intersheetrefs" "${INTERSHEET_REFS}"
-			(at 80.4552 60.96 0)
-			(effects
-				(font
-					(size 1.27 1.27)
-				)
-				(justify left)
-				(hide yes)
-			)
-		)
-	)
 	(global_label "SW1"
 		(shape input)
@@
 	(symbol
 		(lib_id "power:GND")
-		(at 67.31 85.09 90)
+		(at 73.66 60.96 90)
 		(unit 1)
 		(exclude_from_sim no)
@@
 		(fields_autoplaced yes)
 		(property "Reference" "#PWR034"
-			(at 73.66 85.09 0)
+			(at 80.01 60.96 0)
 			(effects
 				(font
@@
 		)
 		(property "Value" "GND"
-			(at 71.12 85.0899 90)
+			(at 77.47 60.9599 90)
 			(effects
 				(font
@@
 		)
 		(property "Footprint" ""
-			(at 67.31 85.09 0)
+			(at 73.66 60.96 0)
 			(effects
 				(font
@@
 		)
 		(property "Datasheet" ""
-			(at 67.31 85.09 0)
+			(at 73.66 60.96 0)
 			(effects
 				(font
@@
 		)
 		(property "Description" "Power symbol creates a global label with name \"GND\" , ground"
-			(at 67.31 85.09 0)
+			(at 73.66 60.96 0)
 			(effects
 				(font
@@
 					(unit 1)
 				)
-			)
-		)
-	)
-	(symbol
-		(lib_id "Jumper:SolderJumper_2_Bridged")
-		(at 63.5 85.09 0)
-		(unit 1)
-		(exclude_from_sim no)
-		(in_bom no)
-		(on_board yes)
-		(dnp no)
-		(fields_autoplaced yes)
-		(property "Reference" "JP1"
-			(at 63.5 78.74 0)
-			(effects
-				(font
-					(size 1.27 1.27)
-				)
-			)
-		)
-		(property "Value" "SolderJumper_2_Bridged"
-			(at 63.5 81.28 0)
-			(effects
-				(font
-					(size 1.27 1.27)
-				)
-			)
-		)
-		(property "Footprint" "Jumper:SolderJumper-2_P1.3mm_Bridged_RoundedPad1.0x1.5mm"
-			(at 63.5 85.09 0)
-			(effects
-				(font
-					(size 1.27 1.27)
-				)
-				(hide yes)
-			)
-		)
-		(property "Datasheet" "~"
-			(at 63.5 85.09 0)
-			(effects
-				(font
-					(size 1.27 1.27)
-				)
-				(hide yes)
-			)
-		)
-		(property "Description" "Solder Jumper, 2-pole, closed/bridged"
-			(at 63.5 85.09 0)
-			(effects
-				(font
-					(size 1.27 1.27)
-				)
-				(hide yes)
-			)
-		)
-		(pin "1"
-		)
-		(pin "2"
-		)
-		(instances
-			(project ""
-				(path "/cc713380-d5d4-4611-b364-320b19da6c16"
-					(reference "JP1")
-					(unit 1)
-				)

Commit message: adjusting foot prints
Parts:
- J1, J2, J3, J4, J5: footprint Connector_PinHeader_2.54mm:PinHeader_1x02_P2.54mm_Vertical -> footprint:PinHeader_1x02_P2.54mm_Vertical
- U3: footprint Seeed Studio XIAO Series Library:XIAO-ESP32C6-SMD -> footprint:XIAO-ESP32C6-SMD
Changed lines of the file:
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@@
 			)
 		)
-		(property "Footprint" "Connector_PinHeader_2.54mm:PinHeader_1x02_P2.54mm_Vertical"
+		(property "Footprint" "footprint:PinHeader_1x02_P2.54mm_Vertical"
 			(at 152.4 124.46 0)
 			(effects
@@
 			)
 		)
-		(property "Footprint" "Connector_PinHeader_2.54mm:PinHeader_1x02_P2.54mm_Vertical"
+		(property "Footprint" "footprint:PinHeader_1x02_P2.54mm_Vertical"
 			(at 228.6 124.46 0)
 			(effects
@@
 			)
 		)
-		(property "Footprint" "Connector_PinHeader_2.54mm:PinHeader_1x02_P2.54mm_Vertical"
+		(property "Footprint" "footprint:PinHeader_1x02_P2.54mm_Vertical"
 			(at 177.8 124.46 0)
 			(effects
@@
 			)
 		)
-		(property "Footprint" "Connector_PinHeader_2.54mm:PinHeader_1x02_P2.54mm_Vertical"
+		(property "Footprint" "footprint:PinHeader_1x02_P2.54mm_Vertical"
 			(at 203.2 124.46 0)
 			(effects
@@
 			)
 		)
-		(property "Footprint" "Seeed Studio XIAO Series Library:XIAO-ESP32C6-SMD"
+		(property "Footprint" "footprint:XIAO-ESP32C6-SMD"
 			(at 162.56 39.37 0)
 			(effects
@@
 			)
 		)
-		(property "Footprint" "Connector_PinHeader_2.54mm:PinHeader_1x02_P2.54mm_Vertical"
+		(property "Footprint" "footprint:PinHeader_1x02_P2.54mm_Vertical"
 			(at 127 124.46 0)
 			(effects
